File: Boston - Current design/PCB/V0.6.1D/Boston-keyboard-V06-1D.kicad_sch (KiCad schematic)
At the start: 594 parts, among them J701 Conn_01x04_MountingPin, J702 Conn_01x03, J705 Conn_01x04_MountingPin, J706 Conn_ARM_JTAG_SWD_10, Q701 DTC123J, Q702 AO4406AL, SW1 MXSwitch, SW10 MXSwitch, SW100 MXSwitch, SW101 MXSwitch, SW102 MXSwitch, SW103 MXSwitch, SW104 MXSwitch, SW105-1 MXSwitch, SW105-2 MXSwitch, SW106 MXSwitch, SW107 MXSwitch, SW108 MXSwitch, SW109 MXSwitch, SW11 MXSwitch, SW110 MXSwitch, SW111 MXSwitch, SW112 MXSwitch, SW113 MXSwitch, SW114 MXSwitch, SW115 MXSwitch, SW116 MXSwitch, SW117 MXSwitch, SW118 MXSwitch, SW119 MXSwitch, SW12 MXSwitch, SW120 MXSwitch, SW121 MXSwitch, SW122 MXSwitch, SW123 MXSwitch, SW124-1 MXSwitch, SW124-2 MXSwitch, SW125 MXSwitch, SW126 Rotary_Encoder_Switch_Chassis, SW127 MXSwitch, SW128 MXSwitch, SW129 MXSwitch, SW13 MXSwitch, SW14 MXSwitch, SW15 MXSwitch, SW16 MXSwitch, SW17 MXSwitch, SW18 MXSwitch, SW19 MXSwitch, SW2 MXSwitch, SW20-1 MXSwitch, SW20-2 MXSwitch, SW200 SW_Push, SW21 MXSwitch, SW22 MXSwitch, SW23 MXSwitch, SW24 MXSwitch, SW25 MXSwitch, SW26 MXSwitch, SW27 MXSwitch, SW28 MXSwitch, SW29 MXSwitch, SW3 MXSwitch, SW30 MXSwitch, SW31 MXSwitch, SW32 MXSwitch, SW33 MXSwitch, SW34 MXSwitch, SW35 MXSwitch, SW36 MXSwitch, SW37 MXSwitch, SW38 MXSwitch, SW39-1 MXSwitch, SW39-2 MXSwitch, SW39-3 MXSwitch, SW4-1 MXSwitch, SW4-2 MXSwitch, SW40 MXSwitch, SW41 MXSwitch, SW42 MXSwitch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

Commit message: Added note that SW123 and SW124-2 were accidentally swapped in the PCB layout
Other:
- note added: "SW123 and SW124-2 were accidentally swapped in the physical PCB layout. The firmware will be changed to reflect this."
