File: Boston - Current design/CNC version/Plate/Hotswap-ANSI/KiCAD files/FR4-hotswap-ANSI-plate.kicad_pcb (KiCad board)
At the start: 2 copper layers, 397 x 159.9 mm, 26 parts

Commit message: Forgot to up the version when fixing the sharp corners
Other:
- board text added: "Boston (Metal Version) - ANSI Hotswap Plate V0.20 - June 27, 2023 Designed by Pylon - open source at http://github.com/bluepylons/Boston"
- board text removed: "Boston (Metal Version) - ANSI Hotswap Plate V0.1 - March 4, 2023 Designed by Pylon - open source at http://github.com/bluepylons/Boston"
Changed lines of the file:
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@@
   (gr_arc (start 247.506249 92.225) (mid 247.359805 92.578571) (end 247.006249 92.725)
     (stroke (width 0.1) (type solid)) (layer "User.2"))
-  (gr_text "Boston (Metal Version) - ANSI Hotswap Plate V0.1 - March 4, 2023\nDesigned by Pylon - open source at http://github.com/bluepylons/Boston" (at 264.318972 14.287512) (layer "B.SilkS")
+  (gr_text "Boston (Metal Version) - ANSI Hotswap Plate V0.20 - June 27, 2023\nDesigned by Pylon - open source at http://github.com/bluepylons/Boston" (at 264.318972 14.287512) (layer "B.SilkS")
     (effects (font (size 1.4 1.4) (thickness 0.3)) (justify left mirror))
   )
